Commit message: included training scripts for all assemblies in a row; Changed the sdf resolution back to 512; Changed Matplotlib Backend to Agg; Copied Franka Gripper Visual s.t. gets found;

File: learning/assets/fabrica/urdf/fabrica_franka/cooling_manifold_4_1.urdf (robot description, URDF)
Before this commit: robot panda, 13 links, 12 joints
Joints:
- joint 4_joint: origin xyz=0.05317573559085994 -0.011758563665637059 0.10659017489333412 rpy=-2.6082377037438773 -0.7558351078688409 2.4308512333224654 -> xyz=-0.03862268248594196 0.011758563664737695 0.14059815221786504 rpy=-3.0592755266364335 -0.15126871699173883 -0.5009188789668045

File: learning/assets/fabrica/urdf/fabrica_franka/cooling_manifold_5_1.urdf (robot description, URDF)
Before this commit: robot panda, 13 links, 12 joints
Joints:
- joint 5_joint: origin xyz=-0.06106503450781084 -0.0071685929262412795 0.1652834637258515 rpy=2.8130989797561035 0.37713132390029647 -0.7467594974543734 -> xyz=0.07947241045123402 0.007168592926170392 0.08210553691265408 rpy=-2.6816488917694232 -0.4989890138044708 2.3389045326528106

File: learning/assets/fabrica/urdf/fabrica_franka/cooling_manifold_6_1.urdf (robot description, URDF)
Before this commit: robot panda, 13 links, 12 joints
Joints:
- joint 6_joint: origin xyz=0.06090687151656282 0.0004219440001332897 0.12070816509733366 rpy=2.9876156677896057 0.15662191053415264 -0.7829017723050925 -> xyz=-0.05766069977058279 -0.0004219440028631616 0.14286509161469502 rpy=-3.010088541152635 -0.13420060104475318 2.3619475250121567
