Commit message: testing an error on "Segmentation fault" while creating the SDF for Assembly "Duct" and "Gamepad". Seems like an VRAM issue, where my 8gb VRAM are not enough?

File: learning/assets/fabrica/urdf/fabrica_franka/gamepad_1_3.urdf (robot description, URDF)
Before this commit: robot panda, 13 links, 12 joints
Joints:
- joint 1_joint: origin xyz=-0.02828292305607283 0.025026232060906872 0.134442037030317 rpy=3.0927041049877153 0.07480211895190436 2.561918185361191 -> xyz=-0.006133972190172213 0.033222080596741616 0.14268245321395082 rpy=-2.8970609777765937 -0.16424051866577116 2.1508583647095008
- joint panda_finger_joint1: origin xyz=0.0 0.015497288691659766 0.0584 rpy=0.0 0.0 0.0 -> xyz=0.0 0.01549726331968439 0.0584 rpy=0.0 0.0 0.0
- joint panda_finger_joint2: origin xyz=0.0 -0.015497288691659766 0.0584 rpy=0.0 0.0 0.0 -> xyz=0.0 -0.01549726331968439 0.0584 rpy=0.0 0.0 0.0

Commit message: trained all assemblies, to be tested

File: learning/assets/fabrica/urdf/fabrica_franka/gamepad_1_3.urdf (robot description, URDF)
Before this commit: robot panda, 13 links, 12 joints
Joints:
- joint 1_joint: origin xyz=-0.006133972190172213 0.033222080596741616 0.14268245321395082 rpy=-2.8970609777765937 -0.16424051866577116 2.1508583647095008 -> xyz=-0.02828292305607283 0.025026232060906872 0.134442037030317 rpy=3.0927041049877153 0.07480211895190436 2.561918185361191
- joint panda_finger_joint1: origin xyz=0.0 0.01549726331968439 0.0584 rpy=0.0 0.0 0.0 -> xyz=0.0 0.015497288691659766 0.0584 rpy=0.0 0.0 0.0
- joint panda_finger_joint2: origin xyz=0.0 -0.01549726331968439 0.0584 rpy=0.0 0.0 0.0 -> xyz=0.0 -0.015497288691659766 0.0584 rpy=0.0 0.0 0.0
